File: PCBs/rev1/rev1.kicad_sch (KiCad schematic)
At the start: 101 parts, among them J1 Conn_02x12, J10 Conn_01x01, J2 Conn_02x12, J3 Conn_02x12, J4 Conn_02x12, J5 Conn_02x12, J6 Conn_02x12, J7 Conn_02x12, J8 Conn_01x03, J9 USB_B_Micro, SW1 SW_Push, U1 RP2040, U2 AZ1117-3.3, U3 W25Q32JVSS, Y1 12Mhz

Commit message: PCB
dhwiqodhiowq
Parts:
- removed J1: Conn_02x12, symbol Connector_Generic:Conn_02x12_Counter_Clockwise
- added J4: Conn_02x12_Odd_Even, Connector_PinHeader_2.54mm:PinHeader_2x12_P2.54mm_Vertical, symbol Connector_Generic:Conn_02x12_Odd_Even
- J1, J10, J11, J7, J8, J9: renamed from J?; footprint (none) -> Connector_PinHeader_2.54mm:PinHeader_1x04_P2.54mm_Vertical
- J12: renamed from J4; footprint (none) -> Connector_PinHeader_2.54mm:PinHeader_2x12_P2.54mm_Vertical; symbol Connector_Generic:Conn_02x12_Counter_Clockwise -> Connector_Generic:Conn_02x12_Odd_Even
- J13: renamed from J5; footprint (none) -> Connector_PinHeader_2.54mm:PinHeader_2x12_P2.54mm_Vertical; symbol Connector_Generic:Conn_02x12_Counter_Clockwise -> Connector_Generic:Conn_02x12_Odd_Even
- J18: renamed from J6; footprint (none) -> Connector_PinHeader_2.54mm:PinHeader_2x12_P2.54mm_Vertical; symbol Connector_Generic:Conn_02x12_Counter_Clockwise -> Connector_Generic:Conn_02x12_Odd_Even
- J19: renamed from J7; footprint (none) -> Connector_PinHeader_2.54mm:PinHeader_2x12_P2.54mm_Vertical; symbol Connector_Generic:Conn_02x12_Counter_Clockwise -> Connector_Generic:Conn_02x12_Odd_Even
- J20: renamed from J?; footprint (none) -> Connector_Phoenix_GMSTB:PhoenixContact_GMSTBA_2,5_4-G_1x04_P7.50mm_Horizontal
- J5: renamed from J2; footprint (none) -> Connector_PinHeader_2.54mm:PinHeader_2x12_P2.54mm_Vertical; symbol Connector_Generic:Conn_02x12_Counter_Clockwise -> Connector_Generic:Conn_02x12_Odd_Even
- J6: renamed from J3; footprint (none) -> Connector_PinHeader_2.54mm:PinHeader_2x12_P2.54mm_Vertical; symbol Connector_Generic:Conn_02x12_Counter_Clockwise -> Connector_Generic:Conn_02x12_Odd_Even
- R1, R10, R13, R14, R15, R16, R17, R20, R21, R22, R23, R24, R25, R26, R27, R28, R29, R30, R31, R32, R33, R34, R35, R36, R37, R38, R39, R40, R41, R42, R43, R44, R45, R46, R7, R8, R9: renamed from R?; footprint (none) -> Resistor_SMD:R_0805_2012Metric
- U1: renamed from U?; footprint (none) -> Package_SO:SO-14_5.3x10.2mm_P1.27mm
- U3: renamed from U?; footprint (none) -> Package_SO:SO-8_5.3x6.2mm_P1.27mm
- gave numbers to parts that had none: 3
- renumbered C3 to C1, C1 to C2, C2 to C3, C5 to C4, C7 to C5, C8 to C6, C4 to C7, C9 to C8, C6 to C9, D2 to D1, D3 to D2, D4 to D3, D5 to D4, D6 to D5, D1 to D6, J10 to J14, J8 to J16, J9 to J2, R2 to R11, R3 to R12, R4 to R18, R5 to R19, R7 to R2, R8 to R3, R9 to R4, R6 to R47, R1 to R48, R11 to R49, R10 to R5, R13 to R50, R12 to R51, R11 to R6, U1 to U4, U3 to U5
Connections:
- net +12V: now also J12.15 (Pin_15), J12.16 (Pin_16), J13.15 (Pin_15), J13.16 (Pin_16), J18.15 (Pin_15), J18.16 (Pin_16), J19.15 (Pin_15), J19.16 (Pin_16), J5.15 (Pin_15), J5.16 (Pin_16), J6.15 (Pin_15), J6.16 (Pin_16), J4.15 (Pin_15), J4.16 (Pin_16); no longer J12.17 (Pin_17), J12.8 (Pin_8), J13.17 (Pin_17), J13.8 (Pin_8), J18.17 (Pin_17), J18.8 (Pin_8), J19.17 (Pin_17), J19.8 (Pin_8), J5.17 (Pin_17), J5.8 (Pin_8), J6.17 (Pin_17), J6.8 (Pin_8)
- net +3V3: now also R1.2, R10.2, R13.2, R14.2, R15.2, R16.2, R17.2, R7.2, R8.2, R9.2
- net +5V: now also J12.10 (Pin_10), J12.9 (Pin_9), J13.10 (Pin_10), J13.9 (Pin_9), J18.10 (Pin_10), J18.9 (Pin_9), J19.10 (Pin_10), J19.9 (Pin_9), J5.10 (Pin_10), J5.9 (Pin_9), J6.10 (Pin_10), J6.9 (Pin_9), J4.10 (Pin_10), J4.9 (Pin_9); no longer J12.20 (Pin_20), J12.5 (Pin_5), J13.20 (Pin_20), J13.5 (Pin_5), J18.20 (Pin_20), J18.5 (Pin_5), J19.20 (Pin_20), J19.5 (Pin_5), J5.20 (Pin_20), J5.5 (Pin_5), J6.20 (Pin_20), J6.5 (Pin_5)
- net -12V: now also J12.13 (Pin_13), J12.14 (Pin_14), J13.13 (Pin_13), J13.14 (Pin_14), J18.13 (Pin_13), J18.14 (Pin_14), J19.13 (Pin_13), J19.14 (Pin_14), J5.13 (Pin_13), J5.14 (Pin_14), J6.13 (Pin_13), J6.14 (Pin_14), J4.13 (Pin_13), J4.14 (Pin_14); no longer J12.18 (Pin_18), J12.7 (Pin_7), J13.18 (Pin_18), J13.7 (Pin_7), J18.18 (Pin_18), J18.7 (Pin_7), J19.18 (Pin_18), J19.7 (Pin_7), J5.18 (Pin_18), J5.7 (Pin_7), J6.18 (Pin_18), J6.7 (Pin_7)
- net A_IN_1: now also J4.19 (Pin_19), J4.20 (Pin_20); no longer J13.10 (Pin_10)
- net A_IN_2: now also J5.19 (Pin_19), J5.20 (Pin_20); no longer J5.10 (Pin_10), J5.15 (Pin_15)
- net A_IN_3: now also J6.19 (Pin_19), J6.20 (Pin_20); no longer J6.10 (Pin_10), J6.15 (Pin_15)
- net A_IN_4: now also J12.19 (Pin_19), J12.20 (Pin_20); no longer J12.10 (Pin_10), J12.15 (Pin_15)
- net A_IN_5: now also J13.19 (Pin_19), J13.20 (Pin_20); no longer J13.15 (Pin_15)
- net A_IN_A: now also J18.19 (Pin_19), J18.20 (Pin_20); no longer J18.10 (Pin_10), J18.15 (Pin_15)
- net A_IN_B: now also J19.19 (Pin_19), J19.20 (Pin_20); no longer J19.10 (Pin_10), J19.15 (Pin_15)
- net A_OUT_L_1: now also J4.23 (Pin_23), J4.24 (Pin_24)
- net A_OUT_L_2: now also J5.23 (Pin_23), J5.24 (Pin_24); no longer J5.12 (Pin_12), J5.13 (Pin_13)
- net A_OUT_L_3: now also J6.23 (Pin_23), J6.24 (Pin_24); no longer J6.12 (Pin_12), J6.13 (Pin_13)
- net A_OUT_L_4: now also J12.23 (Pin_23), J12.24 (Pin_24); no longer J12.12 (Pin_12), J12.13 (Pin_13)
- net A_OUT_L_5: now also J13.23 (Pin_23), J13.24 (Pin_24); no longer J13.12 (Pin_12), J13.13 (Pin_13)
- net A_OUT_L_A: now also J18.23 (Pin_23), J18.24 (Pin_24); no longer J18.12 (Pin_12), J18.13 (Pin_13)
- net A_OUT_L_B: now also J19.23 (Pin_23), J19.24 (Pin_24); no longer J19.12 (Pin_12), J19.13 (Pin_13)
- net A_OUT_R_1: now also J4.21 (Pin_21), J4.22 (Pin_22)
- net A_OUT_R_2: now also J5.21 (Pin_21), J5.22 (Pin_22); no longer J5.11 (Pin_11), J5.14 (Pin_14)
- net A_OUT_R_3: now also J6.21 (Pin_21), J6.22 (Pin_22); no longer J6.11 (Pin_11), J6.14 (Pin_14)
- net A_OUT_R_4: now also J12.21 (Pin_21), J12.22 (Pin_22); no longer J12.11 (Pin_11), J12.14 (Pin_14)
- net A_OUT_R_5: now also J13.21 (Pin_21), J13.22 (Pin_22); no longer J13.11 (Pin_11), J13.14 (Pin_14)
- net A_OUT_R_A: now also J18.21 (Pin_21), J18.22 (Pin_22); no longer J18.11 (Pin_11), J18.14 (Pin_14)
- net A_OUT_R_B: now also J19.21 (Pin_21), J19.22 (Pin_22); no longer J19.11 (Pin_11), J19.14 (Pin_14)
- net DET_1: now also J4.7 (Pin_7), J4.8 (Pin_8); no longer J18.21 (Pin_21)
- net DET_2: now also J5.7 (Pin_7), J5.8 (Pin_8); no longer J5.21 (Pin_21), J5.4 (Pin_4)
- net DET_3: now also J6.7 (Pin_7), J6.8 (Pin_8); no longer J6.21 (Pin_21), J6.4 (Pin_4)
- net DET_4: now also J12.7 (Pin_7), J12.8 (Pin_8); no longer J12.21 (Pin_21), J12.4 (Pin_4)
- net DET_5: now also J13.7 (Pin_7), J13.8 (Pin_8); no longer J13.21 (Pin_21), J13.4 (Pin_4)
- net DET_A: now also J18.7 (Pin_7), J18.8 (Pin_8); no longer J18.4 (Pin_4)
- net DET_B: now also J19.7 (Pin_7), J19.8 (Pin_8); no longer J19.21 (Pin_21), J19.4 (Pin_4)
- net GND: now also J12.11 (Pin_11), J12.12 (Pin_12), J12.17 (Pin_17), J12.18 (Pin_18), J13.11 (Pin_11), J13.12 (Pin_12), J13.17 (Pin_17), J13.18 (Pin_18), J18.11 (Pin_11), J18.12 (Pin_12), J18.17 (Pin_17), J18.18 (Pin_18), J19.11 (Pin_11), J19.12 (Pin_12), J19.17 (Pin_17), J19.18 (Pin_18), J5.11 (Pin_11), J5.12 (Pin_12), J5.17 (Pin_17), J5.18 (Pin_18), J6.11 (Pin_11), J6.12 (Pin_12), J6.17 (Pin_17), J6.18 (Pin_18), J4.11 (Pin_11), J4.12 (Pin_12), J4.17 (Pin_17), J4.18 (Pin_18); no longer J12.16 (Pin_16), J12.19 (Pin_19), J12.6 (Pin_6), J12.9 (Pin_9), J13.16 (Pin_16), J13.19 (Pin_19), J13.6 (Pin_6), J13.9 (Pin_9), J18.16 (Pin_16), J18.19 (Pin_19), J18.6 (Pin_6), J18.9 (Pin_9), J19.16 (Pin_16), J19.19 (Pin_19), J19.6 (Pin_6), J19.9 (Pin_9), J5.16 (Pin_16), J5.19 (Pin_19), J5.6 (Pin_6), J5.9 (Pin_9), J6.16 (Pin_16), J6.19 (Pin_19), J6.6 (Pin_6), J6.9 (Pin_9)
- net GPIO10: now also J6.5 (Pin_5), J6.6 (Pin_6)
- net GPIO11: now also J6.3 (Pin_3), J6.4 (Pin_4)
- net GPIO13: now also J6.2 (Pin_2); no longer J6.24 (Pin_24)
- net GPIO14: now also J12.5 (Pin_5), J12.6 (Pin_6)
- net GPIO15: now also J12.3 (Pin_3), J12.4 (Pin_4)
- net GPIO17: now also J12.2 (Pin_2); no longer J12.24 (Pin_24)
- net GPIO18: now also J13.5 (Pin_5), J13.6 (Pin_6)
- net GPIO19: now also J13.3 (Pin_3), J13.4 (Pin_4)
- net GPIO2: now also J4.5 (Pin_5), J4.6 (Pin_6)
- net GPIO21: now also J13.2 (Pin_2); no longer J13.24 (Pin_24)
- net GPIO3: now also J4.3 (Pin_3), J4.4 (Pin_4)
- net GPIO5: now also J4.1 (Pin_1), J4.2 (Pin_2); no longer J18.24 (Pin_24)
- net GPIO6: now also J5.5 (Pin_5), J5.6 (Pin_6)
- net GPIO7: now also J5.3 (Pin_3), J5.4 (Pin_4)
- net GPIO9: now also J5.2 (Pin_2); no longer J5.24 (Pin_24)
- net SDA_A: now also J18.5 (Pin_5), J18.6 (Pin_6); no longer J18.3 (Pin_3)
- net SDA_B: now also J19.5 (Pin_5), J19.6 (Pin_6); no longer J19.22 (Pin_22), J19.3 (Pin_3)
- net SDL_A: now also J18.3 (Pin_3), J18.4 (Pin_4); no longer J18.2 (Pin_2)
- net SDL_B: now also J19.3 (Pin_3), J19.4 (Pin_4); no longer J19.2 (Pin_2), J19.23 (Pin_23)
- net TRIG_A: now also J18.2 (Pin_2)
- net TRIG_B: now also J19.2 (Pin_2); no longer J19.24 (Pin_24)
- removed net SDA_1: J18.22 (Pin_22), R1.2
- removed net SDA_2: J5.22 (Pin_22), J5.3 (Pin_3), R8.2
- removed net SDA_3: J6.22 (Pin_22), J6.3 (Pin_3), R10.2
- removed net SDA_4: J12.22 (Pin_22), J12.3 (Pin_3), R14.2
- removed net SDA_5: J13.22 (Pin_22), J13.3 (Pin_3), R16.2
- removed net SDL_1: J18.23 (Pin_23), R7.2
- removed net SDL_2: J5.2 (Pin_2), J5.23 (Pin_23), R9.2
- removed net SDL_3: J6.2 (Pin_2), J6.23 (Pin_23), R13.2
- removed net SDL_4: J12.2 (Pin_2), J12.23 (Pin_23), R15.2
- removed net SDL_5: J13.2 (Pin_2), J13.23 (Pin_23), R17.2
- no-connect marks 21 -> 24
Other:
- moved on the sheet: R1, R10, R13, R14, R15, R16, R17, R7, R8, R9
