File: PCBs/rev1/rev1.sch (KiCad schematic (older format))
At the start: 42 parts, among them J1 USB_B_Micro, J2 Conn_01x03, J3 Conn_01x08, J4 Conn_01x05, J5 Conn_01x04, J6 Conn_01x01, SW1 SW_Push, U1 RP2040, U2 AZ1117-3.3, U3 W25Q32JVSS, Y1 12Mhz

Commit message: PCB
dhwiqodhiowq
Parts:
- J1: symbol Connector:USB_B_Micro -> rev1-rescue:USB_B_Micro-Connector
- U1: symbol rp2040:RP2040 -> rev1-rescue:RP2040-rp2040
Changed lines of the file:
@@
 $EndDescr
 $Comp
-L rp2040:RP2040 U1
+L rev1-rescue:RP2040-rp2040 U1
 U 1 1 6168B28C
 P 4800 2250
@@
 $EndComp
 $Comp
-L Connector:USB_B_Micro J1
+L rev1-rescue:USB_B_Micro-Connector J1
 U 1 1 6168F78C
 P 1350 6550
