File: PCBs/ECEN494 KiCAD/FM/FM DRUM/dddd/dddd.kicad_pcb (KiCad board)
At the start: 2 copper layers, 80 x 41.9 mm, 58 parts, among them J1 Conn_02x12_Odd_Even, J2 Conn_01x03, J3 Conn_01x03, J4 Conn_01x03, J5 Conn_01x03, J6 Conn_01x03, J7 Conn_01x03, Q1 2N3904, SW1 SW_DIP_x06, U1 LM555xM, U2 LM555xM, U3 MCP46x2, U4 LM555xM, U5 LM555xM, U6 MCP46x2, U7 MCP46x2, U8 TL072, U9 AD8561

Commit message: k
n
Other:
- net class Default removed
