File: PCBs/ECEN494 KiCAD/HIHAT/Hihat/Hihat.kicad_pcb (KiCad board)
At the start: 2 copper layers, 59.7 x 32.4 mm, 35 parts, among them J1 Conn_02x12_Odd_Even, J2 Conn_01x03, J3 Conn_01x03, Q1 2N3904, Q2 2N3904, Q3 2N3904, SW1 SW_DIP_x02, U7 MCP46x2, U8 TL072

Commit message: k
n
Other:
- net class Default removed
